File: battery_management/battery_management.kicad_pcb (KiCad board)
At the start: 2 copper layers, 90 x 90 mm, 17 parts, among them J1 Conn_02x20_Odd_Even, U1 L7805

Commit message: layout da primeira versao commitado
Other:
- board text added: "ANTARES - 26/04 Gerenciamento energético"
Changed lines of the file:
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@@
-(kicad_pcb (version 20171130) (host pcbnew 5.1.1-8be2ce7~80~ubuntu18.10.1)
+(kicad_pcb (version 20171130) (host pcbnew 5.0.2-bee76a0~70~ubuntu16.04.1)
   (general
     (thickness 1.6)
-    (drawings 12)
+    (drawings 13)
     (tracks 79)
     (zones 0)
@@
   )
   (setup
-    (last_trace_width 3)
+    (last_trace_width 0.25)
     (user_trace_width 1)
     (user_trace_width 3)
@@
     (zone_45_only no)
     (trace_min 0.2)
+    (segment_width 0.2)
+    (edge_width 0.05)
     (via_size 0.8)
     (via_drill 0.4)
@@
     (uvia_min_size 0.2)
     (uvia_min_drill 0.1)
-    (edge_width 0.05)
-    (segment_width 0.2)
     (pcb_text_width 0.3)
     (pcb_text_size 1.5 1.5)
@@
     )
   )
+  (gr_text "ANTARES - 26/04\nGerenciamento energético" (at 135.56 65.07) (layer F.Cu)
+    (effects (font (size 1.5 1.5) (thickness 0.3)))
+  )
   (gr_line (start 115 133) (end 115 57) (layer F.SilkS) (width 0.12))
